File: hardware/panel-usb/kicad/tresvizo-panel-usb.kicad_pcb (KiCad board)
At the start: 4 copper layers, 20.8 x 19.7 mm, 8 parts, among them J501 USB_C, J502 PANEL_USB, U501 USBLC6-2SC6

Commit message: Placa principal v0.2: J404 montado con puente JP101, USB-C de la panel-usb más volado, correcciones de la auditoría y logotipo
- J404 (NTC) se monta de fábrica y la NTC queda opcional. Sin ella, R106 (10 kΩ) va a GND por
  JP101, un puente de soldadura cerrado de fábrica, y el cargador ve 25 °C. Para usar la NTC se
  corta JP101 («cortar JP101» en la serigrafía, sobre el puente). R115 baja junto a R113 para
  dejar sitio a esa línea.
- panel-usb: el canto de la lengüeta retrocede 0.8 mm (v = 0.89) y el USB-C sobresale 1.29 mm; su
  cara sigue a ras de la tapa. El cobre queda a 0.41 mm del canto. En el panel la fresa frente al
  USB-C se ensancha a 3 mm (opción cuts de panelize.py) para dejar 1.71 mm hasta el marco; el
  panel pasa a 82.8 x 79 mm.
- Auditoría: VBUS de J101 al cargador con pistas de 0.8 y 1.0 mm, etiquetas de la batería y del
  NTC separadas, planos internos con 0.12 mm de margen y, en el README, medir el pin 1 de la
  carrier antes de enchufar el arnés y la ranura propuesta en la base bajo J102.
- Logotipo: las piezas con huecos se parten en tiras, porque KiCad deformaba al guardar los
  contornos fracturados (el distintivo de la cara de componentes salía mal).
- ERC 0; DRC con 0 errores, 0 avisos, 0 sin conectar y 0 diferencias de paridad en las dos placas
  y el panel. Comprobación en FreeCAD contra V2.2 sin choques nuevos. Costo estimado de montaje y
  piezas: 213.60 USD por 5 juegos en un panel (J404 suma 2.22 USD), sin el PCB desnudo.
Routing:
- net GND: vias 27 -> 26
Other:
- board size 20.8 x 19.7 mm -> 20.8 x 18.9 mm
