File: hardware/main-board/kicad/gnss.kicad_sch (KiCad schematic)
At the start: 22 parts, among them J301 GNSS, U301 TPS63070RNMR, U302 USBLC6-2SC6, U303 USBLC6-2SC6

Commit message: Placa principal v0.2: build reproducible, J301 en SH 8 y montaje en V2.3 con la carrier real
- Build reproducible: kiid_seed.py siembra los KIID de KiCad en cada paso con el contenido de sus
  entradas (sin las líneas de fecha y ruta de la netlist), y route_rest.py toma del DRC solo qué dos
  islas unir y elige siempre los mismos extremos. Dos builds completos dieron los mismos PCB,
  esquemáticos, BOM, CPL, mapa de pines y Gerber; solo cambian las fechas.
- route_rest.py corta los ciclos de arranque (3 por par de conexiones, 20 por conexión en total),
  guarda lo ruteado antes del relleno de zonas y admite ROUTE_FIRST. build.py rutea primero el bus
  de la microSD: con el WROOM, si otras redes toman antes el paso entre el ESP32, J402 y el zócalo,
  SD_CLK y SD_D2 se quedan sin ruta.
- build.py: PYTHONUNBUFFERED, para que un paso que se cae deje sus últimas líneas, y el error dice
  el script y la señal.
- J301 pasa de GH 8 a SH 8 (SM08B-SRSS-TB, C160407; huella de LCSC con anclajes MP y su modelo):
  ya no se puede cruzar con J101, que es GH 8 y lleva VBUS. Va en v 60.7, con la boca en el canto.
  Suma 2.25 USD a los 5 juegos: 209.11 USD.
- Gerber, vistas y esquema en PDF fuera de git salvo en los hitos (.gitignore y nota en los README).
  El quitado del índice quedó por error en b94647d.
- cad/: STEP regenerados con esta placa (modelos de LCSC corregidos por su .wrl) y placement.json al
  día. Nuevo carrier_bdlx.py: la carrier aproximada con sus componentes, sacada de la foto.
  check_montaje_v2_3.py:
  - mueve la placa desplazamiento_placa_y;
  - prueba también la carrier con componentes: encontró los choques de su USB-C y de las soldaduras
    del arnés, que b94647d corrige;
  - lleva el cable de la 18650 1 mm más adelante junto al riel -X.
- ERC 0. DRC con 0 violaciones, 0 sin conectar y 0 de paridad en la placa, la panel-usb y el panel;
  133 de 133 conexiones. Montaje en V2.3 (b94647d) sin choques paso a paso; el cable de la 18650
  pasa libre, a 0.17 mm como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
Parts:
- J301: footprint tresvizo_lcsc:CONN-SMD_8P-P1.25_XUNPU-WAFER-GH1.25-8PWB -> tresvizo_lcsc:CONN-TH_SM08B-SRSS-TB-LF-SN; LCSC C3029383 -> C160407; MPN WAFER-GH1.25-8PWB -> SM08B-SRSS-TB(LF)(SN)
Changed lines of the file:
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@@
 			)
 		)
-		(property "Footprint" "tresvizo_lcsc:CONN-SMD_8P-P1.25_XUNPU-WAFER-GH1.25-8PWB"
+		(property "Footprint" "tresvizo_lcsc:CONN-TH_SM08B-SRSS-TB-LF-SN"
 			(at 38.1 114.3 0)
 			(effects
@@
 			)
 		)
-		(property "Description" "GH 8 lateral (XUNPU, huella JST SM08B-GHS-TB): 5V, GND, RXD2, TXD2, PPS, EVENT, RESET_N, GND"
+		(property "Description" "SH 8 lateral (JST SM08B-SRSS-TB): 5V, GND, RXD2, TXD2, PPS, EVENT, RESET_N, GND. SH y no GH, para que no se pueda cruzar con J101 (GH 8 con VBUS)"
 			(at 38.1 114.3 0)
 			(effects
@@
 			)
 		)
-		(property "MPN" "WAFER-GH1.25-8PWB"
+		(property "MPN" "SM08B-SRSS-TB(LF)(SN)"
 			(at 38.1 114.3 0)
 			(effects
@@
 			)
 		)
-		(property "LCSC" "C3029383"
+		(property "LCSC" "C160407"
 			(at 38.1 114.3 0)
 			(effects
