File: hardware/main-board/kicad/mcu.kicad_sch (KiCad schematic)
At the start: 18 parts, among them SW201 RESET, SW202 BOOT, U201 ESP32-S3-MINI-1-N4R2

Commit message: Placa principal v0.2: UM980 y BMI088 por cable, conectores hacia cantos o zonas libres, placa panel-usb y un solo panel para JLCPCB
- 46 x 64 mm, 4 capas. El UM980 queda en su carrier BDLX por J301 (GH 8) con 5 V conmutable
  (TPS63070, GPIO45) y el BMI088 vuelve a la tapa por I2C en un segundo bus (J405, GH 7).
- Todos los conectores de cable son GH o SH de 8 pines o menos (kit del propietario), salvo la
  batería (PH 2). Cada uno apunta a un canto o a una zona libre con sitio para la clavija
  enchufada y su cable: áreas de regla clavija_* en el DRC y kicad/plugs.json para el CAD.
- La placa sube 2.5 mm en el tubo (z 23.5-87.5) para que las clavijas del canto inferior tengan
  7.6 mm hasta la base; rieles propuestos en z 39-90 y agujeros nuevos. Comprobada en FreeCAD
  contra V2.2 con modelos 3D y clavijas: sin choques.
- Cargador según el ejemplo de TI: bootstrap junto a sus pines (0.9 y 1.6 mm), salida en abanico
  de la fila inferior y potencia solo por capas externas.
- Placa panel-usb (USB-C a ras de la tapa del panel, GH 8 a J101) y panel de las dos placas con un
  BOM y un CPL (panelize.py, 82.8 x 78 mm).
- Serigrafía sin solapes (silk_clean.py) y logotipo de TresVizo con www.tresvizo.com.
- ERC 0; DRC con 0 errores, 0 avisos, 0 sin conectar y 0 diferencias de paridad en las dos
  placas y el panel. Costo estimado de montaje y piezas: 211 USD por 5 juegos en un panel, sin
  el PCB desnudo.
Connections:
- net ANT_FAULT_N: no longer names the net of U201.37 (IO41)
- net ESP_TX1: no longer names the net of U201.10 (IO6)
- net GNSS_TXD3_MCU renamed GNSS_EVENT_MCU
- net IMU_CS_ACC_N: no longer names the net of U201.19 (IO15)
- net IMU_CS_GYR_N: no longer names the net of U201.20 (IO16)
- net IMU_MISO: no longer names the net of U201.17 (IO13)
- net IMU_MOSI renamed IMU_SDA
- net IMU_SCK renamed IMU_SCL
- no-connect marks 2 -> 7
Changed lines of the file:
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@@
 		(title "ESP32-S3")
 		(date "2026-10-04")
-		(rev "0.1")
+		(rev "0.2")
 		(company "TresVizo")
 		(comment 1 "Exploratorio: no fabricado ni probado")
-		(comment 2 "UM980 + ESP32-S3-MINI-1-N4R2 + BMI088 + BQ25798 (1S; 2S por variante)")
-		(comment 3 "JLCPCB 4 capas JLC04161H-7628, 50 x 76 mm")
+		(comment 2 "ESP32-S3-MINI-1-N4R2 + BQ25798 (1S; 2S por variante); GNSS e IMU por conector")
+		(comment 3 "JLCPCB 4 capas JLC04161H-7628")
 	)
 	(symbol
@@
 		)
 	)
-	(global_label "GNSS_TXD3_MCU"
+	(global_label "GNSS_EVENT_MCU"
 		(shape bidirectional)
 		(at 33.02 54.61 180)
@@
 		)
 	)
-	(wire
-		(pts (xy 35.56 57.15) (xy 33.02 57.15))
-		(stroke
-			(width 0)
-			(type default)
-		)
-	)
-	(global_label "ESP_TX1"
-		(shape bidirectional)
-		(at 33.02 57.15 180)
-		(fields_autoplaced yes)
-		(effects
-			(font
-				(size 1 1)
-			)
-			(justify right)
-		)
-		(property "Intersheetrefs" "${INTERSHEET_REFS}"
-			(at 33.02 57.15 0)
-			(effects
-				(font
-					(size 1 1)
-				)
-				(hide yes)
-			)
-		)
+	(no_connect
+		(at 35.56 57.15)
 	)
 	(wire
@@
 		)
 	)
-	(global_label "IMU_MOSI"
+	(global_label "IMU_SDA"
 		(shape bidirectional)
 		(at 33.02 69.85 180)
@@
 		)
 	)
-	(global_label "IMU_SCK"
+	(global_label "IMU_SCL"
 		(shape bidirectional)
 		(at 33.02 72.39 180)
@@
 		)
 	)
-	(wire
-		(pts (xy 35.56 74.93) (xy 33.02 74.93))
-		(stroke
-			(width 0)
-			(type default)
-		)
-	)
-	(global_label "IMU_MISO"
-		(shape bidirectional)
-		(at 33.02 74.93 180)
-		(fields_autoplaced yes)
-		(effects
-			(font
-				(size 1 1)
-			)
-			(justify right)
-		)
-		(property "Intersheetrefs" "${INTERSHEET_REFS}"
-			(at 33.02 74.93 0)
-			(effects
-				(font
-					(size 1 1)
-				)
-				(hide yes)
-			)
-		)
+	(no_connect
+		(at 35.56 74.93)
 	)
 	(wire
@@
 		)
 	)
-	(wire
-		(pts (xy 35.56 80.01) (xy 33.02 80.01))
-		(stroke
-			(width 0)
-			(type default)
-		)
-	)
-	(global_label "IMU_CS_ACC_N"
-		(shape bidirectional)
-		(at 33.02 80.01 180)
-		(fields_autoplaced yes)
-		(effects
-			(font
-				(size 1 1)
-			)
-			(justify right)
-		)
-		(property "Intersheetrefs" "${INTERSHEET_REFS}"
-			(at 33.02 80.01 0)
-			(effects
-				(font
-					(size 1 1)
-				)
-				(hide yes)
-			)
-		)
-	)
-	(wire
-		(pts (xy 35.56 82.55) (xy 33.02 82.55))
-		(stroke
-			(width 0)
-			(type default)
-		)
-	)
-	(global_label "IMU_CS_GYR_N"
-		(shape bidirectional)
-		(at 33.02 82.55 180)
-		(fields_autoplaced yes)
-		(effects
-			(font
-				(size 1 1)
-			)
-			(justify right)
-		)
-		(property "Intersheetrefs" "${INTERSHEET_REFS}"
-			(at 33.02 82.55 0)
-			(effects
-				(font
-					(size 1 1)
-				)
-				(hide yes)
-			)
-		)
+	(no_connect
+		(at 35.56 80.01)
+	)
+	(no_connect
+		(at 35.56 82.55)
 	)
 	(wire
@@
 		)
 	)
-	(wire
-		(pts (xy 66.04 74.93) (xy 68.58 74.93))
-		(stroke
-			(width 0)
-			(type default)
-		)
-	)
-	(global_label "ANT_FAULT_N"
-		(shape bidirectional)
-		(at 68.58 74.93 0)
-		(fields_autoplaced yes)
-		(effects
-			(font
-				(size 1 1)
-			)
-			(justify left)
-		)
-		(property "Intersheetrefs" "${INTERSHEET_REFS}"
-			(at 68.58 74.93 0)
-			(effects
-				(font
-					(size 1 1)
-				)
-				(hide yes)
-			)
-		)
-	)
-	(wire
+	(no_connect
+		(at 66.04 74.93)
+	)
+	(wire

Commit message: Placa principal v0.2: ESP32-S3-WROOM-1-N16R2 en lugar del MINI-1 y sin LEDs del panel
- U201 = ESP32-S3-WROOM-1-N16R2 (C2913205): 16 MB de flash y 2 MB de PSRAM quad. Huella y
  modelos de LCSC; el .step se corrió 3.65 mm para que coincida con su .wrl y la huella.
- GPIO nuevos para rutear el módulo en la misma placa: microSD CLK 6, CMD 7, D0 5, D1 4, D2 16,
  D3 15 y detección 17; UART del GNSS TX 8 / RX 9; PPS 10, EVENT 11, RESET 12; I2C 13/14;
  IMU 41/42 con INT1 2 e INT3 1; botón 18; puntos de prueba en 35, 36 y 37. README y pinout
  con el mapa para el firmware.
- Fuera J406, sus resistencias y la del STAT del cargador: la carcasa V2.3 no lleva LEDs.
- Misma placa de 46 x 64 mm. H1 pasa a (12.0, 9.6) y el corte del riel +X frente a la antena a
  v 15.1-34.0; antena sin cobre en u 0-6.7, v 15.7-33.7.
- R108 sale de debajo de los pines de la microSD (el ruteador se ciclaba entre SD_D3 y
  CHG_INT_N) y el divisor de TS va bajo L102.
- BUCK_SW y el PGND de U105 prerruteados: la vía que el ruteador ponía junto a L102 hacía caer
  el relleno de zonas de KiCad 10 (-11, también en kicad-cli). route_rest guarda las pistas que
  arranca mientras dura el ruteo.
- DRC 0, sin conexiones pendientes y con paridad en la placa y en el panel; ERC 0. Costo
  estimado 206.86 USD por 5 juegos (montaje + piezas, sin PCB).
- Carcasa V2.3: H1 en z 77.9, riel +X cortado en z 53.7-72.4, placa superior recortada frente
  a la antena y SMA de la carrier con las medidas de la foto. Placa nueva contra la carcasa:
  0 mm3 de choques.
Parts:
- TP203: value IO14 -> IO35
- TP204: value IO42 -> IO36
- TP205: value TXD0 -> IO37
- U201: value ESP32-S3-MINI-1-N4R2 -> ESP32-S3-WROOM-1-N16R2; footprint tresvizo_lcsc:BULETM-SMD_ESP32-S3-MINI-1-N8 -> tresvizo_lcsc:WIRELM-SMD_ESP32-S3-WROOM-1; symbol tresvizo:ESP32-S3-MINI-1_LCSC -> RF_Module:ESP32-S3-WROOM-1; LCSC C3013941 -> C2913205; MPN ESP32-S3-MINI-1-N4R2 -> ESP32-S3-WROOM-1-N16R2
Connections:
- net LED_G is gone; now on net BTN_LED_EN: U201.25 (IO48)
- net LED_R is gone; now on net BTN_SENSE_N: U201.11 (IO18)
- net +3V3: now also U201.2 (3V3); no longer U201.3 (3V3)
- net BTN_LED_EN: no longer U201.33 (IO37)
- net BTN_SENSE_N: no longer U201.14 (IO10)
- net CHG_INT_N: now also U201.23 (IO21); no longer U201.6 (IO2)
- net ESP_BOOT: now also U201.27 (IO0); no longer U201.4 (IO0)
- net ESP_EN: now also U201.3 (EN); no longer U201.45 (EN)
- net ESP_IO3: now also U201.15 (IO3); no longer U201.7 (IO3)
- net FG_ALRT_N: now also U201.24 (IO47); no longer U201.31 (IO35)
- net GND: now also U201.40 (GND), U201.41 (GND); no longer U201.2 (GND), U201.42 (GND), U201.43 (GND), U201.46 (GND), U201.47 (GND), U201.48 (GND), U201.49 (GND), U201.50 (GND), U201.51 (GND), U201.52 (GND), U201.53 (GND), U201.54 (GND), U201.55 (GND), U201.56 (GND), U201.57 (GND), U201.58 (GND), U201.59 (GND), U201.60 (GND), U201.GND
- net GNSS_EVENT_MCU: now also U201.19 (IO11); no longer U201.9 (IO5)
- net GNSS_PPS_MCU: now also U201.18 (IO10); no longer U201.5 (IO1)
- net GNSS_PWR_EN: now also U201.26 (IO45); no longer U201.41 (IO45)
- net GNSS_RESET_MCU: now also U201.20 (IO12); no longer U201.8 (IO4)
- net GNSS_TXD2_MCU: now also U201.17 (IO9); no longer U201.40 (RXD0)
- net I2C_SCL: now also U201.22 (IO14); no longer U201.13 (IO9)
- net I2C_SDA: now also U201.21 (IO13); no longer U201.12 (IO8)
- net IMU_INT1: now also U201.38 (IO2); no longer U201.21 (IO17)
- net IMU_INT3: now also U201.39 (IO1); no longer U201.22 (IO18)
- net IMU_SCL: now also U201.35 (IO42); no longer U201.16 (IO12)
- net IMU_SDA: now also U201.34 (IO41); no longer U201.15 (IO11)
- net SD_CLK: now also U201.6 (IO6); no longer U201.34 (IO38)
- net SD_CMD: now also U201.7 (IO7); no longer U201.29 (IO34)
- net SD_D0: now also U201.5 (IO5); no longer U201.35 (IO39)
- net SD_D1: now also U201.4 (IO4); no longer U201.36 (IO40)
- net SD_D2: now also U201.9 (IO16); no longer U201.27 (IO47)
- net SD_D3: now also U201.8 (IO15); no longer U201.28 (IO33)
- net SD_DET: now also U201.10 (IO17); no longer U201.30 (IO48)
- net USB_DN: now also U201.13 (USB_D-); no longer U201.23 (USB_D-)
- net USB_DP: now also U201.14 (USB_D+); no longer U201.24 (USB_D+)
- net ESP_IO14 renamed ESP_IO35
- net ESP_IO35: now also U201.28 (IO35); no longer U201.18 (IO14)
- net ESP_IO42 renamed ESP_IO36
- net ESP_IO36: now also U201.29 (IO36); no longer U201.38 (IO42)
- net ESP_TX0 renamed ESP_IO37
- net ESP_IO37: now also U201.30 (IO37); no longer U201.39 (TXD0)
- net LED_B: no longer names the net of U201.32 (IO39)
- new net GNSS_TX_MCU: U201.12 (IO8)
- no-connect marks 7 -> 6
Other:
- note added: "ESP32-S3-WROOM-1-N16R2 (16 MB de flash, 2 MB de PSRAM quad)"
- note removed: "ESP32-S3-MINI-1-N4R2 (mismo módulo que la Thing Plus)"
- moved on the sheet: C201, C202, C203, R201, R202, R203, R204, R205, SW201, SW202, TP201, TP202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

Commit message: Placa principal v0.3 compacta: 36 × 71.5 mm para el tubo de Ø52, con USB-C, OLED, botón, LED y BMI088 en la placa
- Rama exploratoria pedida por el propietario el 07-10-2026. Especificación, interfaces con la
  carcasa, colocación y auditoría en research/v03-compacta.md.
- Esquema (ERC 0):
  - USB-C TYPE-C-31-M-12 con Rd de 5.1k, TVS SMF15A y USBLC6;
  - pulsador TS-1187A a BTN_N;
  - LED de estado en GPIO48 con 330 Ω;
  - OLED del propietario soldada sobre pads SMD (J403);
  - BMI088 por I2C (GPIO41/42, INT1 en GPIO2 e INT3 en GPIO1);
  - J102 en GH 4, con dos contactos por polo;
  - TP208 y TP209 en la UART0.
  Fuera J402, J405 y Q402; la panel-usb ya no se usa.
- Placa de 4 capas con muescas para la funda del USB-C y para la clavija SMA de la carrier.
  - Los bloques del cargador y de los reguladores se mueven sin cambiar su geometría interna.
  - La antena del WROOM va hacia −X, con zona sin cobre.
  - Panel de una sola placa.
  - DRC con 0 violaciones, 0 sin conectar y 0 de paridad; el panel, igual.
- Auditoría eléctrica independiente (08-10-2026), con sus siete puntos corregidos:
  - las soldaduras de la OLED ya no quedan frente al SMA de la carrier;
  - puentes del panel lejos del IMU y de los condensadores de potencia;
  - zona sin cobre de la antena más grande;
  - GND de J102 y vías dobles en VPACK;
  - vías junto al pad de tierra del WROOM;
  - LED más brillante;
  - pads de la UART.
- cad/export_board_step.py exporta el STEP en los ejes de la carcasa, con los modelos de LCSC
  corregidos. cad/check_heights.py comprueba los altos contra el tubo: todas las piezas caben con
  0.3 mm de aire.
- Cambios en los scripts:
  - route_rest.py admite límites de búsqueda por entorno;
  - fanout.py respeta las vías prerruteadas;
  - finish_pcb.py --final quita las vías sin uso;
  - cost_jlc.py sirve para una sola placa.
- Costo estimado en JLCPCB: 236.43 USD por 5 placas montadas, sin el PCB ni el envío.
- El build casi siempre se repite igual. En una de cuatro corrid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
Parts:
- added TP208: U0TXD, TestPoint:TestPoint_Pad_D1.0mm, symbol Connector:TestPoint
- added TP209: U0RXD, TestPoint:TestPoint_Pad_D1.0mm, symbol Connector:TestPoint
Connections:
- net ESP_RXD0: now reaches U201.36 (RXD0)
- net ESP_RXD0: now also TP209.1
- net ESP_TXD0: now reaches U201.37 (TXD0)
- net ESP_TXD0: now also TP208.1
- net BTN_LED_EN renamed LED_STATUS
- no-connect marks 6 -> 4
Other:
- moved on the sheet: TP201, TP202, TP203, TP204, TP205, TP206, TP207
