File: hardware/main-board/kicad/power.kicad_sch (KiCad schematic)
At the start: 58 parts, among them J101 PANEL_USB, J102 BATTERY, Q101 AO3400A, Q102 AO3401A, Q103 AO3400A, U101 USBLC6-2SC6, U102 BQ25798RQMR, U103 MAX17048G+T10, U105 TPS62903RPJR, U106 TPS22919DCKR

Commit message: Placa principal v0.2: UM980 y BMI088 por cable, conectores hacia cantos o zonas libres, placa panel-usb y un solo panel para JLCPCB
- 46 x 64 mm, 4 capas. El UM980 queda en su carrier BDLX por J301 (GH 8) con 5 V conmutable
  (TPS63070, GPIO45) y el BMI088 vuelve a la tapa por I2C en un segundo bus (J405, GH 7).
- Todos los conectores de cable son GH o SH de 8 pines o menos (kit del propietario), salvo la
  batería (PH 2). Cada uno apunta a un canto o a una zona libre con sitio para la clavija
  enchufada y su cable: áreas de regla clavija_* en el DRC y kicad/plugs.json para el CAD.
- La placa sube 2.5 mm en el tubo (z 23.5-87.5) para que las clavijas del canto inferior tengan
  7.6 mm hasta la base; rieles propuestos en z 39-90 y agujeros nuevos. Comprobada en FreeCAD
  contra V2.2 con modelos 3D y clavijas: sin choques.
- Cargador según el ejemplo de TI: bootstrap junto a sus pines (0.9 y 1.6 mm), salida en abanico
  de la fila inferior y potencia solo por capas externas.
- Placa panel-usb (USB-C a ras de la tapa del panel, GH 8 a J101) y panel de las dos placas con un
  BOM y un CPL (panelize.py, 82.8 x 78 mm).
- Serigrafía sin solapes (silk_clean.py) y logotipo de TresVizo con www.tresvizo.com.
- ERC 0; DRC con 0 errores, 0 avisos, 0 sin conectar y 0 diferencias de paridad en las dos
  placas y el panel. Costo estimado de montaje y piezas: 211 USD por 5 juegos en un panel, sin
  el PCB desnudo.
Parts:
- removed C121: 100nF, Capacitor_SMD:C_0402_1005Metric, symbol Device:C
- removed C122: 1uF, Capacitor_SMD:C_0402_1005Metric, symbol Device:C
- removed FB101: BLM18PG121SN1D, tresvizo_lcsc:L0603, symbol Device:FerriteBead_Small
- removed R120, R122: 100k, Resistor_SMD:R_0402_1005Metric, symbol Device:R
- removed R121: 22k, Resistor_SMD:R_0402_1005Metric, symbol Device:R
- removed U106: TPS22919DCKR, tresvizo_lcsc:SC-70-6_L2.2-W1.3-P0.65-LS2.1-BR, symbol tresvizo:TPS22919DCK_QOD
- C106, C107: value 10uF -> 22uF; LCSC C15850 -> C45783; MPN CL21A106KAYNNNE -> CL21A226MAQNNNE
- C108, C112, C116: value 10uF -> 100nF; footprint Capacitor_SMD:C_0805_2012Metric -> Capacitor_SMD:C_0402_1005Metric; LCSC C15850 -> C307331; MPN CL21A106KAYNNNE -> CL05B104KB54PNC
- C109, C113: value 100nF -> 22uF; footprint Capacitor_SMD:C_0402_1005Metric -> Capacitor_SMD:C_0805_2012Metric; LCSC C307331 -> C45783; MPN CL05B104KB54PNC -> CL21A226MAQNNNE
- C111: value 22uF -> 10uF; LCSC C45783 -> C15850; MPN CL21A226MAQNNNE -> CL21A106KAYNNNE
- C114, C120: value 22uF -> 100nF; footprint Capacitor_SMD:C_0805_2012Metric -> Capacitor_SMD:C_0402_1005Metric; LCSC C45783 -> C307331; MPN CL21A226MAQNNNE -> CL05B104KB54PNC
- C115: value 100nF -> 10uF; footprint Capacitor_SMD:C_0402_1005Metric -> Capacitor_SMD:C_0805_2012Metric; LCSC C307331 -> C15850; MPN CL05B104KB54PNC -> CL21A106KAYNNNE
- C117: value 100nF -> 47nF; footprint Capacitor_SMD:C_0402_1005Metric -> Capacitor_SMD:C_0603_1608Metric; LCSC C307331 -> C1622; MPN CL05B104KB54PNC -> CL10B473KB8NNNC
- C118: value 47nF -> 22uF; footprint Capacitor_SMD:C_0603_1608Metric -> Capacitor_SMD:C_0805_2012Metric; LCSC C1622 -> C45783; MPN CL10B473KB8NNNC -> CL21A226MAQNNNE
- D101: value SMF20A -> SMF15A; footprint tresvizo_lcsc:SOD-123F_L2.8-W1.8-LS3.7-RD -> tresvizo_lcsc:SOD-123FL_L2.7-W1.8-LS3.8-RD; LCSC C123788 -> C19077509; MPN SMF20A -> SMF15A
- J101: footprint tresvizo_lcsc:CONN-SMD_6P-P2.00_B6B-PH-SM4-TB-LF-SN -> tresvizo_lcsc:CONN-SMD_8P-P1.25_XUNPU-WAFER-GH1.25-8PWB; symbol Connector_Generic_MountingPin:Conn_01x06_MountingPin -> Connector_Generic_MountingPin:Conn_01x08_MountingPin; LCSC C471518 -> C3029383; MPN B6B-PH-SM4-TB(LF)(SN) -> WAFER-GH1.25-8PWB
- R101, R117: value 0 -> 10k; LCSC C17168 -> C25744; MPN 0402WGF0000TCE -> 0402WGF1002TCE; now fitted
- R102: value 0 -> 22k; LCSC C17168 -> C25768; MPN 0402WGF0000TCE -> 0402WGF2202TCE; now fitted
- R103: value 10k -> 4.7k; LCSC C25744 -> C25900; MPN 0402WGF1002TCE -> 0402WGF4701TCE
- R104: value 22k -> 5.1k; LCSC C25768 -> C25905; MPN 0402WGF2202TCE -> 0402WGF5101TCE
- R105: value 4.7k -> 30k; footprint Resistor_SMD:R_0402_1005Metric -> Resistor_SMD:R_0603_1608Metric; LCSC C25900 -> C22984; MPN 0402WGF4701TCE -> 0603WAF3002T5E
- R106: value 5.1k -> 10k; LCSC C25905 -> C25744; MPN 0402WGF5101TCE -> 0402WGF1002TCE
- R107: value 30k -> 100; footprint Resistor_SMD:R_0603_1608Metric -> Resistor_SMD:R_0402_1005Metric; LCSC C22984 -> C25076; MPN 0603WAF3002T5E -> 0402WGF1000TCE
- R109: value 100 -> 1k; LCSC C25076 -> C11702; MPN 0402WGF1000TCE -> 0402WGF1001TCE
- R110: value 10k -> 1M; LCSC C25744 -> C26083; MPN 0402WGF1002TCE -> 0402WGF1004TCE
- R111: value 1k -> 100k; LCSC C11702 -> C25741; MPN 0402WGF1001TCE -> 0402WGF1003TCE
- R113: value 100k -> 0; LCSC C25741 -> C17168; MPN 0402WGF1003TCE -> 0402WGF0000TCE
- R114: value 1M -> 10k; LCSC C26083 -> C25744; MPN 0402WGF1004TCE -> 0402WGF1002TCE
- R115: now not fitted
- R116, R119: value 10k -> 22k; LCSC C25744 -> C25768; MPN 0402WGF1002TCE -> 0402WGF2202TCE
- R118: value 22k -> 100k; LCSC C25768 -> C25741; MPN 0402WGF2202TCE -> 0402WGF1003TCE
Connections:
- net +3V3: now also C118.1, R108.1, R114.1, R115.1, R118.1; no longer R110.1, R116.1, R117.1
- net BATREV_G: now also R110.2; no longer R112.2
- net BATREV_SENSE: now also R111.2, R112.1; no longer R113.2, R114.1
- net BUCK_EN: now also R116.2, R117.1; no longer R118.2, R119.1
- net BUCK_FB: now also R118.2, R119.1
- net BUCK_SS: now also C117.1; no longer C118.1
- net CHG_BATP: now also R107.2; no longer R109.2
- net CHG_ILIM: now also R101.2, R102.1; no longer R103.2, R104.1
- net CHG_INT_N: now also R108.2; no longer R110.2
- net CHG_LED_K: now also R109.2; no longer R111.2
- net CHG_PROG: now also R103.1; no longer R105.1
- net CHG_STAT: now also R109.1; no longer R111.1
- net CHG_TS: now also R104.2, R105.1, R106.1; no longer R106.2, R107.1, R108.1
- net FG_ALRT_N: now also R114.2; no longer R116.2
- net FG_VDD: now also C114.1, R113.2; no longer C115.1, R117.2
- net GND: now also J101.4 (Pin_4), J101.5 (Pin_5), R102.2, R103.2, R106.2, R112.2, R117.2; no longer J101.3 (Pin_3), R104.2, R107.2, R108.2, R114.2
- net PMID: no longer C109.1
- net REGN: now also R101.1, R104.1; no longer R103.1, R106.1
- net USB_DN: now also J101.7 (Pin_7); no longer J101.4 (Pin_4), R102.1
- net USB_DP: now also J101.8 (Pin_8); no longer J101.5 (Pin_5), R101.1
- net VBATT_IN: now also R111.1; no longer R113.1
- net VBAT_CHG: now also C113.1; no longer C114.1
- net VBUS: now also J101.3 (Pin_3)
- net VPACK: now also R107.1, R110.1, R113.1; no longer R109.1, R112.1, R115.1
- net VSYS: now also C109.1, C115.1, R116.1; no longer C113.1, C117.1, R118.1
- net CHG_DN: no longer names the net of U102.7 (D-)
- net CHG_DN: no longer R102.2
- net CHG_DP: no longer names the net of U102.6 (D+)
- net CHG_DP: no longer R101.2
- no-connect marks 1 -> 3
Other:
- note removed: "Riel conmutado del UM980"
- moved on the sheet: C101, C102, C103, C104, C105, C106, C107, C108, C109, C110, C111, C112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

Commit message: Placa principal v0.2: J404 montado con puente JP101, USB-C de la panel-usb más volado, correcciones de la auditoría y logotipo
- J404 (NTC) se monta de fábrica y la NTC queda opcional. Sin ella, R106 (10 kΩ) va a GND por
  JP101, un puente de soldadura cerrado de fábrica, y el cargador ve 25 °C. Para usar la NTC se
  corta JP101 («cortar JP101» en la serigrafía, sobre el puente). R115 baja junto a R113 para
  dejar sitio a esa línea.
- panel-usb: el canto de la lengüeta retrocede 0.8 mm (v = 0.89) y el USB-C sobresale 1.29 mm; su
  cara sigue a ras de la tapa. El cobre queda a 0.41 mm del canto. En el panel la fresa frente al
  USB-C se ensancha a 3 mm (opción cuts de panelize.py) para dejar 1.71 mm hasta el marco; el
  panel pasa a 82.8 x 79 mm.
- Auditoría: VBUS de J101 al cargador con pistas de 0.8 y 1.0 mm, etiquetas de la batería y del
  NTC separadas, planos internos con 0.12 mm de margen y, en el README, medir el pin 1 de la
  carrier antes de enchufar el arnés y la ranura propuesta en la base bajo J102.
- Logotipo: las piezas con huecos se parten en tiras, porque KiCad deformaba al guardar los
  contornos fracturados (el distintivo de la cara de componentes salía mal).
- ERC 0; DRC con 0 errores, 0 avisos, 0 sin conectar y 0 diferencias de paridad en las dos placas
  y el panel. Comprobación en FreeCAD contra V2.2 sin choques nuevos. Costo estimado de montaje y
  piezas: 213.60 USD por 5 juegos en un panel (J404 suma 2.22 USD), sin el PCB desnudo.
Parts:
- added JP101: NTC_CORTAR, tresvizo_lcsc:SolderJumper-2_P1.3mm_Bridged_RoundedPad1.0x1.5mm, symbol Jumper:SolderJumper_2_Bridged
Connections:
- net GND: now also JP101.2 (B); no longer R106.2
- new net CHG_TS_FIJA: JP101.1 (A), R106.2
Other:
- moved on the sheet: C114, J102, Q101, Q102, Q103, R106, R107, R108, R109, R110, R111, R112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

Commit message: Placa principal v0.2: techo de entrada del USB a ~1.45 A (R102 22k -> 8.2k)
Revisión del propietario: con ILIM en 10k/22k el cargador podía pedir ~2.9 A a cualquier puerto,
sin detectar cuánto da. Con 10k/8.2k desde REGN (4.6-5.0 V) el techo queda en 1.34-1.56 A, que
alcanza para cargar 1S a 1 A con el equipo encendido. La variante 2S vuelve a 22k (~2.9 A).
Solo cambia el valor de R102 (C25924): pistas y gerbers de cobre iguales; ERC 0, DRC 0 en la
placa y en el panel, paridad 0.

README: queda para v0.3 la detección por CC del USB-C y el par diferencial D+/D-, que pide
invertir los pines 7/8 de J101 y J502. En Full Speed la diferencia de largo actual (9 mm, unos
60 ps) no afecta.
Parts:
- R102: value 22k -> 8.2k; LCSC C25768 -> C25924; MPN 0402WGF2202TCE -> 0402WGF8201TCE
Changed lines of the file:
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@@
 			)
 		)
-		(property "Value" "22k"
+		(property "Value" "8.2k"
 			(at 182.88 105.264 270)
 			(effects
@@
 			)
 		)
-		(property "MPN" "0402WGF2202TCE"
+		(property "MPN" "0402WGF8201TCE"
 			(at 186.69 106.68 0)
 			(effects
@@
 			)
 		)
-		(property "LCSC" "C25768"
+		(property "LCSC" "C25924"
 			(at 186.69 106.68 0)
 			(effects

Commit message: Placa principal v0.2: ESP32-S3-WROOM-1-N16R2 en lugar del MINI-1 y sin LEDs del panel
- U201 = ESP32-S3-WROOM-1-N16R2 (C2913205): 16 MB de flash y 2 MB de PSRAM quad. Huella y
  modelos de LCSC; el .step se corrió 3.65 mm para que coincida con su .wrl y la huella.
- GPIO nuevos para rutear el módulo en la misma placa: microSD CLK 6, CMD 7, D0 5, D1 4, D2 16,
  D3 15 y detección 17; UART del GNSS TX 8 / RX 9; PPS 10, EVENT 11, RESET 12; I2C 13/14;
  IMU 41/42 con INT1 2 e INT3 1; botón 18; puntos de prueba en 35, 36 y 37. README y pinout
  con el mapa para el firmware.
- Fuera J406, sus resistencias y la del STAT del cargador: la carcasa V2.3 no lleva LEDs.
- Misma placa de 46 x 64 mm. H1 pasa a (12.0, 9.6) y el corte del riel +X frente a la antena a
  v 15.1-34.0; antena sin cobre en u 0-6.7, v 15.7-33.7.
- R108 sale de debajo de los pines de la microSD (el ruteador se ciclaba entre SD_D3 y
  CHG_INT_N) y el divisor de TS va bajo L102.
- BUCK_SW y el PGND de U105 prerruteados: la vía que el ruteador ponía junto a L102 hacía caer
  el relleno de zonas de KiCad 10 (-11, también en kicad-cli). route_rest guarda las pistas que
  arranca mientras dura el ruteo.
- DRC 0, sin conexiones pendientes y con paridad en la placa y en el panel; ERC 0. Costo
  estimado 206.86 USD por 5 juegos (montaje + piezas, sin PCB).
- Carcasa V2.3: H1 en z 77.9, riel +X cortado en z 53.7-72.4, placa superior recortada frente
  a la antena y SMA de la carrier con las medidas de la foto. Placa nueva contra la carcasa:
  0 mm3 de choques.
Parts:
- removed R119: 22k, Resistor_SMD:R_0402_1005Metric, symbol Device:R
- R109: value 1k -> 1M; LCSC C11702 -> C26083; MPN 0402WGF1001TCE -> 0402WGF1004TCE
- R110: value 1M -> 100k; LCSC C26083 -> C25741; MPN 0402WGF1004TCE -> 0402WGF1003TCE
- R111: value 100k -> 1M; LCSC C25741 -> C26083; MPN 0402WGF1003TCE -> 0402WGF1004TCE
- R112: value 1M -> 0; LCSC C26083 -> C17168; MPN 0402WGF1004TCE -> 0402WGF0000TCE
- R113: value 0 -> 10k; LCSC C17168 -> C25744; MPN 0402WGF0000TCE -> 0402WGF1002TCE
- R114: value 10k -> 0; LCSC C25744 -> C17168; MPN 0402WGF1002TCE -> 0402WGF0000TCE; now not fitted
- R115: value 0 -> 22k; LCSC C17168 -> C25768; MPN 0402WGF0000TCE -> 0402WGF2202TCE; now fitted
- R116: value 22k -> 10k; LCSC C25768 -> C25744; MPN 0402WGF2202TCE -> 0402WGF1002TCE
- R117: value 10k -> 100k; LCSC C25744 -> C25741; MPN 0402WGF1002TCE -> 0402WGF1003TCE
- R118: value 100k -> 22k; LCSC C25741 -> C25768; MPN 0402WGF1003TCE -> 0402WGF2202TCE
Connections:
- net CHG_LED_K is gone; now on net BATREV_G: R109.2
- net +3V3: now also R113.1, R117.1; no longer R115.1, R118.1
- net BATREV_G: no longer R110.2
- net BATREV_SENSE: now also R110.2, R111.1; no longer R111.2, R112.1
- net BUCK_EN: now also R115.2, R116.1; no longer R116.2, R117.1
- net BUCK_FB: now also R117.2, R118.1; no longer R118.2
- net FG_ALRT_N: now also R113.2; no longer R114.2
- net FG_VDD: now also R112.2, R114.2; no longer R113.2, R115.2
- net GND: now also R111.2, R116.2, R118.2; no longer R112.2, R117.2
- net VBATT_IN: now also R110.1; no longer R111.1
- net VPACK: now also R109.1, R112.1; no longer R110.1, R113.1
- net VSYS: now also R115.1; no longer R116.1
- net CHG_STAT: no longer names the net of U102.1 (STAT)
- net CHG_STAT: no longer R109.1
- no-connect marks 3 -> 4
Other:
- moved on the sheet: R109, R110, R111, R112, R113, R116, R117, R118
Changed lines of the file:
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@@
 		(company "TresVizo")
 		(comment 1 "Exploratorio: no fabricado ni probado")
-		(comment 2 "ESP32-S3-MINI-1-N4R2 + BQ25798 (1S; 2S por variante); GNSS e IMU por conector")
+		(comment 2 "ESP32-S3-WROOM-1-N16R2 + BQ25798 (1S; 2S por variante); GNSS e IMU por conector")
 		(comment 3 "JLCPCB 4 capas JLC04161H-7628")
 	)
@@
 		)
 	)
-	(wire
-		(pts (xy 133.35 62.23) (xy 135.89 62.23))
-		(stroke
-			(width 0)
-			(type default)
-		)
-	)
-	(label "CHG_STAT"
-		(at 135.89 62.23 0)
-		(fields_autoplaced yes)
-		(effects
-			(font
-				(size 1 1)
-			)
-			(justify left bottom)
-		)
+	(no_connect
+		(at 133.35 62.23)
 	)
 	(wire
@@
 			)
 		)
-		(property "Description" "ILIM_HIZ: con 22k da ~2.9 A de techo de entrada"
+		(property "Description" "ILIM_HIZ: con 8.2k da ~1.45 A de techo de entrada (1S); 22k da ~2.9 A (2S)"
 			(at 148.59 106.68 0)
 			(effects
@@
 	)
 	(symbol
-		(lib_id "Device:R")
-		(at 255.27 137.16 90)
-		(unit 1)
-		(exclude_from_sim no)
-		(in_bom yes)
-		(on_board yes)
-		(dnp no)
-		(property "Reference" "R109"
-			(at 251.46 134.144 270)
-			(effects
-				(font
-					(size 1.27 1.27)
-				)
-				(justify left bottom)
-			)
-		)
-		(property "Value" "1k"
-			(at 251.46 135.744 270)
-			(effects
-				(font
-					(size 1 1)
-				)
-				(justify left bottom)
-			)
-		)
-		(property "Footprint" "Resistor_SMD:R_0402_1005Metric"
-			(at 255.27 137.16 0)
-			(effects
-				(font
-					(size 1.27 1.27)
-				)
-				(hide yes)
-			)
-		)
-		(property "Datasheet" ""
-			(at 255.27 137.16 0)
-			(effects
-				(font
-					(size 1.27 1.27)
-				)
-				(hide yes)
-			)
-		)
-		(property "Description" "LED de carga del panel (ánodo a +3V3)"
-			(at 255.27 137.16 0)
-			(effects
-				(font
-					(size 1.27 1.27)
-				)
-				(hide yes)
-			)
-		)
-		(property "MPN" "0402WGF1001TCE"
-			(at 255.27 137.16 0)
-			(effects
-				(font
-					(size 1.27 1.27)
-				)
-				(hide yes)
-			)
-		)
-		(property "LCSC" "C11702"
-			(at 255.27 137.16 0)
-			(effects
-				(font
-					(size 1.27 1.27)
-				)
-				(hide yes)
-			)
-		)
-		(pin "1"
-		)
-		(pin "2"
-		)
-		(instances
-			(project "tresvizo-main"
-				(path "/9a83bcba-5afe-57b6-aafc-7b297421890f/e680a61f-2584-5531-b79e-1aca3f5bfe2f"
-					(reference "R109")
-					(unit 1)
-				)
-			)
-		)
-	)
-	(wire
-		(pts (xy 251.46 137.16) (xy 248.92 137.16))
-		(stroke
-			(width 0)
-			(type default)
-		)
-	)
-	(label "CHG_STAT"
-		(at 248.92 137.16 180)
-		(fields_autoplaced yes)
-		(effects
-			(font
-				(size 1 1)
-			)
-			(justify right bottom)
-		)
-	)
-	(wire
-		(pts (xy 259.08 137.16) (xy 261.62 137.16))
-		(stroke
-			(width 0)
-			(type default)
-		)
-	)
-	(global_label "CHG_LED_K"
-		(shape bidirectional)
-		(at 261.62 137.16 0)
-		(fields_autoplaced yes)
-		(effects
-			(font
-				(size 1 1)
-			)
-			(justify left)
-		)
-		(property "Intersheetrefs" "${INTERSHEET_REFS}"
-			(at 261.62 137.16 0)
-			(effects
-				(font
-					(size 1 1)
-				)
-				(hide yes)
-			)
-		)
-	)
-	(symbol
 		(lib_id "Transistor_FET:AO3400A")
 		(at 341.63 40.64 0)
@@
 		(on_board yes)
 		(dnp no)
-		(property "Reference" "R110"
+		(property "Reference" "R109"
 			(at 384.81 27.464 270)
 			(effects
@@
 			(project "tresvizo-main"
 				(path "/9a83bcba-5afe-57b6-aafc-7b297421890f/e680a61f-2584-5531-b79e-1aca3f5bfe2f"
-					(reference "R110")
+					(reference "R109")
 					(unit 1)
 				)
@@
 		(on_board yes)
 		(dnp no)
-		(property "Reference" "R111"
+		(property "Reference" "R110"
 			(at 452.12 27.464 270)
 			(effects
@@
 			(project "tresvizo-main"
 				(path "/9a83bcba-5afe-57b6-aafc-7b297421890f/e680a61f-2584-5531-b79e-1aca3f5bfe2f"
-					(reference "R111")
+					(reference "R110")
 					(unit 1)
 				)
@@
 		(on_board yes)
 		(dnp no)
-		(property "Reference" "R112"
+		(property "Reference" "R111"
 			(at 499.11 27.464 270)
 			(effects
@@
 			(project "tresvizo-main"
 				(path "/9a83bcba-5afe-57b6-aafc-7b297421890f/e680a61f-2584-5531-b79e-1aca3f5bfe2f"
-					(reference "R112")
+					(reference "R111")
 					(unit 1)
 				)
@@
 		(on_board yes)
 		(dnp no)
-		(property "Reference" "R113"
+		(property "Reference" "R112"
 			(at 417.83 64.294 270)
 			(effects
@@
 			(project "tresvizo-main"
 				(path "/9a83bcba-5afe-57b6-aafc-7b297421890f/e680a61f-2584-5531-b79e-1aca3f5bfe2f"
-					(reference "R113")
+					(reference "R112")
 					(unit 1)
 				)
@@
 		(on_board yes)
 		(dnp no)
-		(property "Reference" "R114"
+		(property "Reference" "R113"
 			(at 445.77 64.294 270)
 			(effects
@@
 			(project "tresvizo-main"
 				(path "/9a83bcba-5afe-57b6-aafc-7b297421890f/e680a61f-2584-5531-b79e-1aca3f5bfe2f"
-					(reference "R114")
+					(reference "R113")
 					(unit 1)
 				)
@@
 		(on_board yes)
 		(dnp yes)
-		(property "Reference" "R115"
+		(property "Reference" "R114"
 			(at 477.52 64.294 270)
 			(effects
@@
 			(project "tresvizo-main"
 				(path "/9a83bcba-5afe-57b6-aafc-7b297421890f/e680a61f-2584-5531-b79e-1aca3f5bfe2f"
-					(reference "R115")
+					(reference "R114")
 					(unit 1)
 				)
@@
 		(on_board yes)
 		(dnp no)
-		(property "Reference" "R116"
+		(property "Reference" "R115"
 			(at 92.71 160.814 270)
 			(effects
@@
 			(project "tresvizo-main"
 				(path "/9a83bcba-5afe-57b6-aafc-7b297421890f/e680a61f-2584-5531-b79e-1aca3f5bfe2f"
-					(reference "R116")
+					(reference "R115")
 					(unit 1)
 				)
@@
 		(on_board yes)
 		(dnp no)
-		(property "Reference" "R117"
+		(property "Reference" "R116"
 			(at 128.27 160.814 270)
 			(effects
@@
 			(project "tresvizo-main"
 				(path "/9a83bcba-5afe-57b6-aafc-7b297421890f/e680a61f-2584-5531-b79e-1aca3f5bfe2f"
-					(reference "R117")
+					(reference "R116")
 					(unit 1)
 				)
@@
 		(on_board yes)
 		(dnp no)
-		(property "Reference" "R118"
+		(property "Reference" "R117"
 			(at 50.8 191.294 270)
 			(effects
@@
 			(project "tresvizo-main"
 				(path "/9a83bcba-5afe-57b6-aafc-7b297421890f/e680a61f-2584-5531-b79e-1aca3f5bfe2f"
-					(reference "R118")
+					(reference "R117")
 					(unit 1)
 				)
@@
 		(on_board yes)
 		(dnp no)
-		(property "Reference" "R119"
+		(property "Reference" "R118"
 			(at 86.36 191.294 270)
 			(effects
@@
 			(project "tresvizo-main"
 				(path "/9a83bcba-5afe-57b6-aafc-7b297421890f/e680a61f-2584-5531-b79e-1aca3f5bfe2f"
-					(reference "R119")
+					(reference "R118")
 					(unit 1)
 				)
