File: hardware/main-board/kicad/io.kicad_sch (KiCad schematic)
At the start: 24 parts, among them J401 TF-015, J403 OLED, J404 NTC, Q401 AO3401A, SW401 BOTON, U401 BMI088

Commit message: v0.3: OLED con VCC en el pin 1 y microSD en su posición real, con muesca de 8
Placa v0.3:
- J403 pasa a VCC, GND, SCL, SDA, que es lo que dice la foto del anuncio del módulo del
  propietario (Mercado Libre, ANPOMNHBUK). Antes era GND, VCC: la OLED habría recibido la
  alimentación invertida. Antes de pedir hay que confirmarlo en la serigrafía de la unidad.
- El anuncio da el controlador SSD1315, compatible con las bibliotecas del SSD1306: queda en la
  tabla del firmware.
- Placa rehecha con build.py: ERC 0, DRC 0/0/0 y panel 0/0. Cambia el ruteo; la colocación no.
- Plano de LCD wiki de la OLED (MC096) comparado con el del vendedor: coinciden en vidrio,
  agujeros y PCB, y da los espesores (PCB 1.2, vidrio 1.5).

Carcasa V3.0:
- Posición de la tarjeta según la hoja de SOFNG del TF-015 (LCSC C113206), desde la boca de J401:
  trabada asoma 2.50 (x 19.0, antes x 17.5 en el modelo), se empuja hasta 1.32 para soltarla y
  expulsada asoma 5.60. En la muesca, la trabada queda 0.4 bajo la cara de fuera y la expulsada
  sobresale 2.7.
- Muesca para la uña de 5 a 8 mm, para que entre la yema.
- El cuerpo de TPU de la tapa en la ranura empieza en r 26.0: queda a 0.54 del canto de la
  tarjeta trabada, así cerrar la tapa no la empuja (el zócalo es de empuje).
- check_v3_0.py: la tarjeta trabada va en su ranura con el ajuste guiado de 0.3, como la funda
  del USB-C, y no cuenta como aire a piezas compradas.
- Comprobación con el STEP real de la placa: 0 choques en posición final y en los 11 barridos,
  guarda de pared sin faltantes y objetivos B1, B2, B3 y B7 cumplidos.

Pendiente: confirmar el orden de los pines en la OLED real, probar impresa la muesca y la tapa
de puertos, medir el pack, la carrier y los agujeros de la OLED, y confirmar el conector de la
antena.
Connections:
- net +3V3: now also J403.1 (Pin_1); no longer J403.2 (Pin_2)
- net GND: now also J403.2 (Pin_2); no longer J403.1 (Pin_1)
Other:
- note added: "J403 (OLED del propietario, soldada a mano): antes de pedir, comprobar en la serigrafía del módulo el orden de GND y VCC (aquí: +3V3, GND, I2C_SCL, I2C_SDA)."
- note removed: "J403 (OLED del propietario, soldada a mano): antes de pedir, comprobar en la serigrafía del módulo el orden de GND y VCC (aquí: GND, +3V3, I2C_SCL, I2C_SDA)."
Changed lines of the file:
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@@
 			)
 		)
-		(property "Description" "Módulo OLED 0.96 in I2C de 4 pines del propietario (no va en el montaje de JLCPCB): 1 GND, 2 +3V3, 3 I2C_SCL, 4 I2C_SDA; pin 1 = el de la izquierda mirado de frente con los pines arriba"
+		(property "Description" "Módulo OLED 0.96 in I2C de 4 pines del propietario (no va en el montaje de JLCPCB): 1 +3V3, 2 GND, 3 I2C_SCL, 4 I2C_SDA; pin 1 = el de la izquierda mirado de frente con los pines arriba"
 			(at 182.88 120.65 0)
 			(effects
@@
 	)
 	(symbol
-		(lib_id "power:GND")
-		(at 175.26 118.11 270)
+		(lib_id "power:+3V3")
+		(at 175.26 118.11 90)
 		(unit 1)
 		(exclude_from_sim no)
@@
 			)
 		)
-		(property "Value" "GND"
-			(at 175.26 121.31 90)
-			(effects
-				(font
-					(size 1 1)
-				)
-				(hide yes)
+		(property "Value" "+3V3"
+			(at 175.26 114.91 270)
+			(effects
+				(font
+					(size 1 1)
+				)
 			)
 		)
@@
 	)
 	(symbol
-		(lib_id "power:+3V3")
-		(at 175.26 120.65 90)
+		(lib_id "power:GND")
+		(at 175.26 120.65 270)
 		(unit 1)
 		(exclude_from_sim no)
@@
 			)
 		)
-		(property "Value" "+3V3"
-			(at 175.26 117.45 270)
-			(effects
-				(font
-					(size 1 1)
-				)
+		(property "Value" "GND"
+			(at 175.26 123.85 90)
+			(effects
+				(font
+					(size 1 1)
+				)
+				(hide yes)
 			)
 		)
@@
 		)
 	)
-	(text "J403 (OLED del propietario, soldada a mano): antes de pedir, comprobar en la serigrafía del módulo el orden de GND y VCC (aquí: GND, +3V3, I2C_SCL, I2C_SDA)."
+	(text "J403 (OLED del propietario, soldada a mano): antes de pedir, comprobar en la serigrafía del módulo el orden de GND y VCC (aquí: +3V3, GND, I2C_SCL, I2C_SDA)."
 		(exclude_from_sim no)
 		(at 12.7 161.29 0)
